File: TI/TI_Adapter.kicad_pcb (KiCad board)
At the start: 2 copper layers, 22 x 16 mm, 4 parts, among them P1 TI_JTAG, P3 TI_jtag

Commit message: Updated layouts
Routing:
- added copper zone on B.Cu, net /TI_GND
- added copper zone on F.Cu, net /TI_GND
Changed lines of the file:
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@@
     (links 14)
     (no_connects 0)
-    (area 103.924999 62.924999 126.176191 79.075001)
+    (area 93.150001 57.3 126.176191 79.075001)
     (thickness 1.6)
     (drawings 6)
@@
   (segment (start 124.9172 70.8152) (end 124.9172 74.9996) (width 0.25) (layer F.Cu) (net 9))
   (segment (start 124.6632 70.5612) (end 124.9172 70.8152) (width 0.25) (layer F.Cu) (net 9))
+  (zone (net 4) (net_name /TI_GND) (layer F.Cu) (hatch edge 0.508)
+    (connect_pads (clearance 0.508))
+    (min_thickness 0.254)
+    (fill yes (arc_segments 16) (thermal_gap 0.508) (thermal_bridge_width 0.508))
+    (polygon
+      (pts
+        (xy 126 79) (xy 104 79) (xy 104 63) (xy 126 63)
+      )
+    )
+  )
+  (zone (net 4) (net_name /TI_GND) (layer B.Cu) (hatch edge 0.508)
+    (connect_pads (clearance 0.508))
+    (min_thickness 0.254)
+    (fill yes (arc_segments 16) (thermal_gap 0.508) (thermal_bridge_width 0.508))
+    (polygon
+      (pts
+        (xy 126 79) (xy 104 79) (xy 104 63) (xy 126 63)
+      )
+    )
+  )
 )
